File: TapType_MainPCB/TapType.kicad_sch (KiCad schematic)
At the start: 36 parts, among them J1 USB_C_Receptacle_USB2.0_16P, J2 Conn_01x06, J3 Conn_01x06, J4 Conn_01x06, J5 Conn_01x06, J6 Conn_01x06, Q1 SS8050, Q2 SS8050, SW1 SW_SPST, SW2 SW_SPST, U1 ESP32-S3-WROOM-1, U2 USBLC6-2P6, U3 DRV2605LDGS, U6 CP2102N-A02-GQFN28

Commit message: Finished KICAD files + Photos
Parts:
- added C1, C2, C5: 1uF, Capacitor_SMD:C_0603_1608Metric, symbol Device:C
- added C15, C6: 100nF, Capacitor_SMD:C_0603_1608Metric, symbol Device:C
- added C16: 22uF, Capacitor_SMD:C_0603_1608Metric, symbol Device:C
- added C3, C4: 4.7uF, Capacitor_SMD:C_0603_1608Metric, symbol Device:C
- added D1, D2, D3, D7: SML-E12P8WT86, Diode_SMD:D_0603_1608Metric, symbol Device:LED
- added D4: SZBZX84C6V2ET1G, easyeda2kicad:SOD-123_L2.7-W1.6-LS3.7-RD, symbol Device:D_Zener
- added D5: SMF5.0A, Diode_SMD:D_SOD-123F, symbol Device:D_Zener
- added J1: JST S2B-PH-K-S-GW, easyeda2kicad:CONN-TH_S2B-PH-K-S-GW, symbol Connector_Generic:Conn_01x02
- added JP1, JP2, JP3: SolderJumper_3_Open, Jumper:SolderJumper-3_P2.0mm_Open_TrianglePad1.0x1.5mm, symbol Jumper:SolderJumper_3_Open
- added JP4: SolderJumper_2_Open, Jumper:SolderJumper-2_P1.3mm_Open_TrianglePad1.0x1.5mm, symbol Jumper:SolderJumper_2_Open
- added MOTOR_N_STRAIN_RELIEF1, MOTOR_P_STRAIN_RELIEF1: TestPoint, strain_relief:strain relief, symbol Connector:TestPoint
- added Q1: IRLML6402TRPBF, Package_TO_SOT_SMD:SOT-23, symbol Transistor_FET:IRLML6402
- added R1, R2: 1.5k, Resistor_SMD:R_0603_1608Metric, symbol Device:R
- added R20, R4, R5, R6: 220R, Resistor_SMD:R_0603_1608Metric, symbol Device:R
- added R3, R8: 10k, Resistor_SMD:R_0603_1608Metric, symbol Device:R
- added R7: 100k, Resistor_SMD:R_0603_1608Metric, symbol Device:R
- added S1: MSK12C02, easyeda2kicad:SW-SMD_G-SWITCH_MK-12C02-G015, symbol MSK12C02:MSK12C02
- added U1: BQ24074RGT, Package_DFN_QFN:VQFN-16-1EP_3x3mm_P0.5mm_EP1.6x1.6mm, symbol Battery_Management:BQ24074RGT
- added U2: AP2112K-3.3, Package_TO_SOT_SMD:SOT-23-5, symbol Regulator_Linear:AP2112K-3.3
- added U3: MAX17048G_T10, MAX17048G_T10:SON50P200X200X80-9N, symbol MAX17048G_T10:MAX17048G_T10
- added U6: USBLC6-2P6, Package_TO_SOT_SMD:SOT-666, symbol Power_Protection:USBLC6-2P6
- C10: renamed from C5; footprint (none) -> Capacitor_SMD:C_0603_1608Metric
- C11: renamed from C6; footprint (none) -> Capacitor_SMD:C_0603_1608Metric
- C12: renamed from C1; value C -> 100nF; footprint (none) -> Capacitor_SMD:C_0603_1608Metric
- C13: renamed from C7; footprint (none) -> Capacitor_SMD:C_0603_1608Metric
- C14: renamed from C8; footprint (none) -> Capacitor_SMD:C_0603_1608Metric
- C7: renamed from C2; footprint (none) -> Capacitor_SMD:C_0603_1608Metric
- C8: renamed from C3; footprint (none) -> Capacitor_SMD:C_0603_1608Metric
- C9: renamed from C4; footprint (none) -> Capacitor_SMD:C_0603_1608Metric
- D6: renamed from D1; footprint (none) -> Diode_SMD:D_0603_1608Metric
- J2: renamed from J1; footprint (none) -> easyeda2kicad:TYPE-C-SMD_SBC-160S1A-20-S412
- J3: renamed from J2; footprint (none) -> easyeda2kicad:FPC-SMD_6P-P0.50_FPC-05FB-6PH20
- J4: renamed from J3; footprint (none) -> easyeda2kicad:FPC-SMD_6P-P0.50_FPC-05FB-6PH20
- J5: renamed from J4; footprint (none) -> easyeda2kicad:FPC-SMD_6P-P0.50_FPC-05FB-6PH20
- J6: renamed from J5; footprint (none) -> easyeda2kicad:FPC-SMD_6P-P0.50_FPC-05FB-6PH20
- J7: renamed from J6; footprint (none) -> easyeda2kicad:FPC-SMD_6P-P0.50_FPC-05FB-6PH20
- MOTOR_N_PAD1: renamed from MOTOR_N_PAD; footprint (none) -> TestPoint:TestPoint_Pad_D2.0mm
- MOTOR_P_PAD1: renamed from MOTOR_P_PAD; footprint (none) -> TestPoint:TestPoint_Pad_D2.0mm
- R10: renamed from R8; footprint (none) -> Resistor_SMD:R_0603_1608Metric
- R11: renamed from R6; footprint (none) -> Resistor_SMD:R_0603_1608Metric
- R12: renamed from R3; footprint (none) -> Resistor_SMD:R_0603_1608Metric
- R13: renamed from R9; footprint (none) -> Resistor_SMD:R_0603_1608Metric
- R14: renamed from R10; footprint (none) -> Resistor_SMD:R_0603_1608Metric
- R15: renamed from R4; footprint (none) -> Resistor_SMD:R_0603_1608Metric
- R16: renamed from R2; footprint (none) -> Resistor_SMD:R_0603_1608Metric
- R17: renamed from R1; footprint (none) -> Resistor_SMD:R_0603_1608Metric
- R18: renamed from R12; footprint (none) -> Resistor_SMD:R_0603_1608Metric
- R19: renamed from R11; footprint (none) -> Resistor_SMD:R_0603_1608Metric
- R9: renamed from R7; footprint (none) -> Resistor_SMD:R_0603_1608Metric
- SW1: renamed from SW2; footprint (none) -> easyeda2kicad:KEY-SMD_B3U-1000PM
- SW2: renamed from SW1; footprint (none) -> easyeda2kicad:KEY-SMD_B3U-1000PM
- renumbered Q1 to Q2, Q2 to Q3, U2 to U4, U6 to U5, U3 to U7, U1 to U8
Connections:
- net +3.3V: now also J3.6 (Pin_6), C15.1, C16.1, C5.1, R8.2, U2.5 (VOUT); no longer J3.1 (Pin_1)
- net GND: now also J3.2 (Pin_2), C1.2, C15.2, C16.2, C2.2, C3.2, C4.2, C5.2, C6.2, D3.1 (K), D5.2 (A), D7.1 (K), J1.2 (Pin_2), JP1.1 (A), JP2.1 (A), R1.2, R2.2, R3.2, R7.2, S1.4_1 (GND), S1.4_2 (GND), S1.4_3 (GND), S1.4_4 (GND), U1.17 (VSS), U1.4 (~{CE}), U1.8 (VSS), U2.2 (GND), U3.1 (CTG), U3.4 (GND), U3.6 (QSTRT), U3.9 (EP), U6.2 (GND); no longer J3.5 (Pin_5)
- net IMU1_INT: now also J3.1 (Pin_1), U8.25 (IO48); no longer J3.6 (Pin_6), U8.22 (IO14)
- net IMU1_SA0: now also J3.3 (Pin_3), U8.24 (IO47); no longer J3.4 (Pin_4), U8.4 (IO4)
- net IMU2_INT: now also U8.10 (IO17); no longer U8.8 (IO15)
- net IMU2_SA0: now also U8.11 (IO18); no longer U8.5 (IO5)
- net IMU3_INT: now also U8.8 (IO15); no longer U8.9 (IO16)
- net IMU3_SA0: now also U8.9 (IO16); no longer U8.6 (IO6)
- net IMU4_INT: now also U8.6 (IO6); no longer U8.10 (IO17)
- net IMU5_INT: now also U8.4 (IO4); no longer U8.11 (IO18)
- net IMU5_SA0: now also U8.5 (IO5); no longer U8.38 (IO2)
- net MOTOR_TRIG: now also U8.23 (IO21); no longer U8.39 (IO1)
- net SCL: now also J3.4 (Pin_4), U3.7 (SCL), U6.3 (I/O2), U6.4 (I/O2); no longer J3.3 (Pin_3)
- net SDA: now also J3.5 (Pin_5), U8.18 (IO10), U3.8 (SDA), U6.1 (I/O1), U6.6 (I/O1); no longer J3.2 (Pin_2), U8.12 (IO8)
- net VBUS: now also C1.1, JP1.3 (B), JP2.3 (B), U1.13 (IN)
- net ALERT: now reaches U8.21 (IO13)
- net ALERT: now also R8.1, U3.5 (~{ALERT})
- new net: D7.2 (A), R20.1
- new net: R20.2, U8.12 (IO8)
- new net: D4.1 (A), Q1.1 (G), R7.1
- new net: D2.2 (A), R5.1
- new net: JP2.2 (C), U1.5 (EN2)
- new net: D2.1 (K), U1.9 (~{CHG})
- new net: C2.1, JP3.2 (C), U2.1 (VIN), U2.3 (EN)
- new net: D5.1 (K), JP4.1 (A), Q1.3 (D), S1.2
- new net: J1.1 (Pin_1), S1.3
- new net: R3.1, U1.1 (TS)
- new net: R1.1, U1.12 (ILIM)
- new net: R2.1, U1.16 (ISET)
- new net: JP1.2 (C), U1.6 (EN1)
- new net: D1.1 (K), U1.7 (~{PGOOD})
- new net: D1.2 (A), R4.1
- new net: D3.2 (A), R6.1
- new net VCC: C4.1, JP3.3 (B), R4.2, R5.2, U1.10 (OUT), U1.11 (OUT)
- new net V_BATT: C3.1, C6.1, D4.3 (K), JP3.1 (A), JP4.2 (B), Q1.2 (S), R6.2, U1.2 (BAT), U1.3 (BAT), U3.2 (CELL), U3.3 (VDD)
- no-connect marks 22 -> 42
Other:
- note added: "Double check J1 footprint"
- note added: "ITERM left unconnected to set termination current to default 10% termination threshold EN1/EN2 is used to select charge current. Do not let them unconnected. EN2 EN1 0 0 - 100mA -> use this 0 1 - 500mA 1 0 - ILIM (mA) OUT : 4.4V I_IN_MAX = 1550 / 1500 = 1.033 A ≈ 1.03 A I_CHG_FAST = 890 / 1500 = 0.593 A ≈ 593 mA"
- note added: "What are the PSRAM pins for? What is GPIO16 used for? (ROMM boot-log printing on UART)"
- note added: "low battery threshold is programmable via the CONFIG register (ATHD bits)"
- note added: "motor wire strain relief"
- note added: "this trace need to handle charge current (100mA/500mA)"
- moved on the sheet: D6, R12, R15, R16, R19
